File: Eagle-Tutorial-1-Files/blinky.sch (EAGLE design)
At the start: 10 parts, among them IC1 LM555D

Commit message: doc(sch) add a description frame
Other:
- note added: "NE555 projet to test Eagle"
Changed lines of the file:
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@@
 <?xml version="1.0" encoding="utf-8"?>
 <!DOCTYPE eagle SYSTEM "eagle.dtd">
-<eagle version="6.2">
+<eagle version="8.7.0">
 <drawing>
 <settings>
 <setting alwaysvectorfont="no"/>
+<setting keepoldvectorfont="yes"/>
 <setting verticaltext="up"/>
 </settings>
@@
 <part name="P+4" library="supply1" deviceset="VCC" device=""/>
 <part name="P+5" library="supply1" deviceset="VCC" device=""/>
+<part name="FRAME1" library="frames" library_urn="urn:adsk.eagle:library:229" deviceset="DINA5_L" device=""/>
 </parts>
 <sheets>
 <sheet>
 <plain>
+<text x="53.34" y="-10.16" size="1.778" layer="106">NE555 projet to test Eagle</text>
 </plain>
 <instances>
@@
 <instance part="P+4" gate="VCC" x="25.4" y="35.56" rot="R90"/>
 <instance part="P+5" gate="VCC" x="58.42" y="27.94"/>
+<instance part="FRAME1" gate="G$1" x="-35.56" y="-30.48"/>
 </instances>
 <busses>
@@
 </schematic>
 </drawing>
+<compatibility>
+<note version="8.2" severity="warning">
+Since Version 8.2, EAGLE supports online libraries. The ids
+of those online libraries will not be understood (or retained)
+with this version.
+</note>
+<note version="8.3" severity="warning">
+Since Version 8.3, EAGLE supports URNs for individual library
+assets (packages, symbols, and devices). The URNs of those assets
+will not be understood (or retained) with this version.
+</note>
+</compatibility>
 </eagle>
